File: kicad/pong/pong.kicad_pcb (KiCad board)
At the start: 2 copper layers, 34 parts, among them J1 VIDEO OUT, J2 POWER INPUT, Q1 2N3904, Q2 2N3904, SW1 RESET, SW2 CONFIG, SW4 GAME SELECT, U1 AY-3-8500, U2 4072

Commit message: Terminada
Parts:
- added REF**: Pin_D0.7mm_L6.5mm_W1.8mm_FlatFork, Connector_Pin:Pin_D0.7mm_L6.5mm_W1.8mm_FlatFork, F.Cu at (98.4, 62.7)
- added REF**: Pin_D0.7mm_L6.5mm_W1.8mm_FlatFork, Connector_Pin:Pin_D0.7mm_L6.5mm_W1.8mm_FlatFork, F.Cu at (98.7, 59.6)
- added REF**: Pin_D0.7mm_L6.5mm_W1.8mm_FlatFork, Connector_Pin:Pin_D0.7mm_L6.5mm_W1.8mm_FlatFork, F.Cu at (84.7, 77.9)
- added REF**: Pin_D0.7mm_L6.5mm_W1.8mm_FlatFork, Connector_Pin:Pin_D0.7mm_L6.5mm_W1.8mm_FlatFork, F.Cu at (84.7, 84.4)
- added REF**: Pin_D0.7mm_L6.5mm_W1.8mm_FlatFork, Connector_Pin:Pin_D0.7mm_L6.5mm_W1.8mm_FlatFork, F.Cu at (80.3, 83.6)
- added REF**: Pin_D0.7mm_L6.5mm_W1.8mm_FlatFork, Connector_Pin:Pin_D0.7mm_L6.5mm_W1.8mm_FlatFork, F.Cu at (80.3, 80.2)
- added REF**: Pin_D0.7mm_L6.5mm_W1.8mm_FlatFork, Connector_Pin:Pin_D0.7mm_L6.5mm_W1.8mm_FlatFork, F.Cu at (90.3, 58.1)
- added REF**: Pin_D0.7mm_L6.5mm_W1.8mm_FlatFork, Connector_Pin:Pin_D0.7mm_L6.5mm_W1.8mm_FlatFork, F.Cu at (90.3, 65.6)
- C1, C2, C3, C4, C5, C6: footprint Capacitor_THT:C_Rect_L4.0mm_W2.5mm_P2.50mm -> Capacitor_THT:C_Disc_D3.8mm_W2.6mm_P2.50mm
- J1: footprint w_conn_av:rca_white -> Connector_av:rca_white
- LS1: footprint Buzzer_Beeper:MagneticBuzzer_ProSignal_ABI-010-RC -> Connector_PinHeader_2.00mm:PinHeader_1x02_P2.00mm_Horizontal
- RV1, RV2: footprint Potentiometer_THT:Potentiometer_Alps_RK09K_Single_Horizontal -> Connector_PinHeader_2.00mm:PinHeader_1x03_P2.00mm_Horizontal
- SW4: footprint Connector_PinHeader_1.00mm:PinHeader_1x05_P1.00mm_Horizontal -> Connector_PinHeader_2.00mm:PinHeader_1x05_P2.00mm_Horizontal
- moved RV2 93.6 mm to (55.0, 47.0), turned to 90 degrees
- moved R5 78.7 mm to (108.7, 59.7), turned to 270 degrees
- moved R11 75.2 mm to (71.5, 49.4)
- moved R4 74.2 mm to (105.8, 67.3), turned to 90 degrees
- moved R8 63.9 mm to (111.8, 67.3), turned to 90 degrees
- moved J1 61.7 mm to (110.6, 80.9)
- moved J2 57.3 mm to (108.3, 54.8), turned to 180 degrees
- moved C7 53.0 mm to (113.9, 72.3), turned to 180 degrees
- moved C5 45.3 mm to (88.6, 46.4), turned to 180 degrees
- moved RV1 45.1 mm to (63.2, 47.0)
- moved C1 39.2 mm to (56.5, 81.5), turned to 0 degrees
- moved R2 36.5 mm to (55.8, 84.6), turned to 0 degrees
- moved C3 29.7 mm to (81.4, 46.4), turned to 0 degrees
- moved LS1 21.6 mm to (56.9, 79.0), turned to 180 degrees
- moved R10 21.5 mm to (71.5, 46.4), turned to 0 degrees
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Routing:
- net VCC: track 14.6 -> 196.9 mm, vias 0 -> 2
- net GND: track 124.1 -> 205.7 mm, vias 0 -> 2
- net Net-(C1-Pad1): track 5.79 -> 44.6 mm, vias 0 -> 2
- net Net-(C5-Pad1): track 0.00 -> 27.6 mm
- net Net-(U1-Pad24): track 82.3 -> 62.3 mm
- net Net-(C3-Pad1): track 0.00 -> 19.3 mm
- net Net-(U1-Pad6): track 66.6 -> 49.7 mm
- net Net-(LS1-Pad2): track 62.3 -> 46.4 mm
- net Net-(J1-Pad1): track 0.00 -> 15.1 mm
- net Net-(R11-Pad1): track 0.00 -> 13.4 mm
- net Net-(C4-Pad1): track 0.00 -> 12.5 mm
- net Net-(R3-Pad1): track 3.30 -> 15.1 mm
- net Net-(R4-Pad1): track 0.00 -> 11.3 mm
- net Net-(D1-Pad2): track 10.5 -> 20.0 mm
- net Net-(SW4-Pad2): track 6.05 -> 15.2 mm
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Other:
- board outline added: 63.5 x 47.8 mm
