File: kicad/pong/pong.sch (KiCad schematic (older format))
At the start: 34 parts, among them J1 VIDEO OUT, J2 POWER INPUT, Q1 2N3904, Q2 2N3904, SW1 RESET, SW4 GAME SELECT, U1 AY-3-8500, U2 4072

Commit message: Terminada
Parts:
- C1, C2, C3, C4, C5, C6: footprint Capacitor_THT:C_Rect_L4.0mm_W2.5mm_P2.50mm -> Capacitor_THT:C_Disc_D3.8mm_W2.6mm_P2.50mm
- J1: footprint w_conn_av:rca_white -> Connector_av:rca_white
- LS1: footprint Buzzer_Beeper:MagneticBuzzer_ProSignal_ABI-010-RC -> Connector_PinHeader_2.00mm:PinHeader_1x02_P2.00mm_Horizontal
- RV1, RV2: footprint Potentiometer_THT:Potentiometer_Alps_RK09K_Single_Horizontal -> Connector_PinHeader_2.00mm:PinHeader_1x03_P2.00mm_Horizontal
- SW2: renamed from SW?; footprint (none) -> Button_Switch_THT:SW_DIP_SPSTx04_Slide_9.78x12.34mm_W7.62mm_P2.54mm
- SW4: footprint Connector_PinHeader_1.00mm:PinHeader_1x05_P1.00mm_Horizontal -> Connector_PinHeader_2.00mm:PinHeader_1x05_P2.00mm_Horizontal
Other:
- note added: "01/07/2019"
- note added: "Black and White Implementation"
- moved on the sheet: C1, C2, C3, C4, C5, C6, C7, D1, D2, J1, J2, L1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
